File: mohawk/soundChip.kicad_sch (KiCad schematic)
At the start: 17 parts, among them U5 TLV320AIC3204IRHBR

Commit message: clean up traces; add missing serial resistors for I²S lines
Parts:
- added R16, R17, R18, R19: 27, Resistor_SMD:R_0805_2012Metric, symbol Device:R_Small
- R15: value 0 -> 10
Connections:
- net GPIO18/PCM.CLK: now also R17.2; no longer U5.2 (BCLK)
- net GPIO19/PCM.FS: now also R16.2; no longer U5.3 (WCLK)
- net GPIO20/PCM.DIN: now also R19.2; no longer U5.5 (DOUT_MFP2)
- net GPIO21/PCM.DOUT: now also R18.2; no longer U5.4 (DIN_MFP1)
- new net: R17.1, U5.2 (BCLK)
- new net: R16.1, U5.3 (WCLK)
- new net: R18.1, U5.4 (DIN_MFP1)
- new net: R19.1, U5.5 (DOUT_MFP2)
Other:
- moved on the sheet: R15
