File: mohawk/mohawk.kicad_sch (KiCad schematic)
At the start: 29 parts, among them J1 GPIO, J2 SMA, J3 UI Header, J4 DB9 Header, U1 CAT24C256, U2 SC16IS752IPW_128, U4 MAX232, Y1 ASE-1.8432MHz

Commit message: more routing clean up; add external power solder pads, add Makefile
Parts:
- added J5: +5V In, mohawk:SolderWirePad 1x02, symbol Connector_Generic:Conn_01x02
Connections:
- net +5V: now also J5.1 (Pin_1)
- net GND: now also J5.2 (Pin_2)

Commit message: add test points for EXT_UART; add 3d model for oscillator
Parts:
- added TP1: TX, TestPoint:TestPoint_Pad_D1.0mm, symbol Connector:TestPoint
- added TP2: RTS, TestPoint:TestPoint_Pad_D1.0mm, symbol Connector:TestPoint
- added TP3: RX, TestPoint:TestPoint_Pad_D1.0mm, symbol Connector:TestPoint
- added TP4: CTS, TestPoint:TestPoint_Pad_D1.0mm, symbol Connector:TestPoint
- added TP5: GND, TestPoint:TestPoint_Pad_D1.0mm, symbol Connector:TestPoint
- C2: value 4.7µF -> 100nF
- R6: value 0 -> 1k
Connections:
- net EXT_UART_CTS: now also TP4.1
- net EXT_UART_RTS: now also TP2.1
- net EXT_UART_RX: now also TP3.1
- net EXT_UART_TX: now also TP1.1
- net GND: now also TP5.1
Other:
- note added: "External Power Solder Pads"
- moved on the sheet: J5
